Commit message: Add gnss link

File: f1eighth_sensor_kit_description/urdf/sensor_kit.xacro (robot description, xacro)
@@ -50,6 +50,13 @@
       <child link="imu_link"/>
     </joint>
+    <link name="imu_link">
+      <inertial>
+        <mass value="0.1"/>
+        <origin xyz="0 0 0"/>
+        <inertia ixx="0.1" ixy="0" ixz="0" iyy="0.1" iyz="0" izz="0.1"/>
+      </inertial>
+    </link>
     <!-- gnss -->
-    <!-- <joint name="gnss_joint" type="fixed">
+    <joint name="gnss_joint" type="fixed">
       <origin
         xyz="${calibration['sensor_kit_base_link']['gnss_base_link']['x']}
@@ -62,5 +69,12 @@
       <parent link="sensor_kit_base_link"/>
       <child link="gnss_base_link"/>
-    </joint>  -->
+    </joint>
+    <link name="gnss_base_link">
+      <inertial>
+        <mass value="0.1"/>
+        <origin xyz="0 0 0"/>
+        <inertia ixx="0.1" ixy="0" ixz="0" iyy="0.1" iyz="0" izz="0.1"/>
+      </inertial>
+    </link>
     <!-- camera -->
     <joint name="zedxm_camera_joint" type="fixed">
