Commit message: Add LiDAR frames to sensor_kit.xacro.

File: autosdv_sensor_kit_description/urdf/sensor_kit.xacro (robot description, xacro)
@@ -4,6 +4,7 @@
     <xacro:include filename="$(find zed_wrapper)/urdf/zed_macro.urdf.xacro"/>
     <xacro:include filename="$(find imu_description)/urdf/imu.xacro"/>
+    <xacro:include filename="$(find blickfeld_driver)/config/blickfeld_cube1.xacro"/>
     <xacro:arg name="gpu" default="false"/>
-    <xacro:arg name="config_dir" default="$(find autosdv_sensor_kit_description)/config"/>
+    <xacro:arg name="config_dir" default="$(find autosdv_sensor_kit_description)/config"/>b
     <xacro:property name="sensor_kit_base_link" default="sensor_kit_base_link"/>
     <joint name="${sensor_kit_base_link}_joint" type="fixed">
@@ -17,18 +18,58 @@
     <!-- sensor -->
     <xacro:property name="calibration" value="${xacro.load_yaml('$(arg config_dir)/sensor_kit_calibration.yaml')}"/>
-    <!-- lidar -->
-    <joint name="lidar_joint" type="fixed">
+    <!-- Blickfeld Cube 1 LiDAR -->
+    <joint name="cube1_joint" type="fixed">
       <origin
-        xyz="${calibration['sensor_kit_base_link']['lidar']['x']}
-             ${calibration['sensor_kit_base_link']['lidar']['y']}
-             ${calibration['sensor_kit_base_link']['lidar']['z']}"
-        rpy="${calibration['sensor_kit_base_link']['lidar']['roll']}
-             ${calibration['sensor_kit_base_link']['lidar']['pitch']}
-             ${calibration['sensor_kit_base_link']['lidar']['yaw']}"
+        xyz="${calibration['sensor_kit_base_link']['cube1']['x']}
+             ${calibration['sensor_kit_base_link']['cube1']['y']}
+             ${calibration['sensor_kit_base_link']['cube1']['z']}"
+        rpy="${calibration['sensor_kit_base_link']['cube1']['roll']}
+             ${calibration['sensor_kit_base_link']['cube1']['pitch']}
+             ${calibration['sensor_kit_base_link']['cube1']['yaw']}"
       />
       <parent link="sensor_kit_base_link"/>
-      <child link="lidar"/>
+      <child link="cube1"/>
     </joint>
-    <link name="lidar">
+    <link name="cube1">
+      <inertial>
+        <mass value="0.1"/>
+        <origin xyz="0 0 0"/>
+        <inertia ixx="0.1" ixy="0" ixz="0" iyy="0.1" iyz="0" izz="0.1"/>
+      </inertial>
+    </link>
+    <!-- Velodyne VLP-32C LiDAR -->
+    <joint name="vlp32c_joint" type="fixed">
+      <origin
+        xyz="${calibration['sensor_kit_base_link']['vlp32c']['x']}
+             ${calibration['sensor_kit_base_link']['vlp32c']['y']}
+             ${calibration['sensor_kit_base_link']['vlp32c']['z']}"
+        rpy="${calibration['sensor_kit_base_link']['vlp32c']['roll']}
+             ${calibration['sensor_kit_base_link']['vlp32c']['pitch']}
+             ${calibration['sensor_kit_base_link']['vlp32c']['yaw']}"
+      />
+      <parent link="sensor_kit_base_link"/>
+      <child link="vlp32c"/>
+    </joint>
+    <link name="vlp32c">
+      <inertial>
+        <mass value="0.1"/>
+        <origin xyz="0 0 0"/>
+        <inertia ixx="0.1" ixy="0" ixz="0" iyy="0.1" iyz="0" izz="0.1"/>
+      </inertial>
+    </link>
+    <!-- Seyond Robin-W LiDAR -->
+    <joint name="robin_w_joint" type="fixed">
+      <origin
+        xyz="${calibration['sensor_kit_base_link']['robin_w']['x']}
+             ${calibration['sensor_kit_base_link']['robin_w']['y']}
+             ${calibration['sensor_kit_base_link']['robin_w']['z']}"
+        rpy="${calibration['sensor_kit_base_link']['robin_w']['roll']}
+             ${calibration['sensor_kit_base_link']['robin_w']['pitch']}
+             ${calibration['sensor_kit_base_link']['robin_w']['yaw']}"
+      />
+      <parent link="sensor_kit_base_link"/>
+      <child link="robin_w"/>
+    </joint>
+    <link name="robin_w">
       <inertial>
         <mass value="0.1"/>

Commit message: Add 4 USB cameras support.

File: autosdv_sensor_kit_description/urdf/sensor_kit.xacro (robot description, xacro)
@@ -6,5 +6,5 @@
     <xacro:include filename="$(find blickfeld_driver)/config/blickfeld_cube1.xacro"/>
     <xacro:arg name="gpu" default="false"/>
-    <xacro:arg name="config_dir" default="$(find autosdv_sensor_kit_description)/config"/>b
+    <xacro:arg name="config_dir" default="$(find individual_params)/config/default/autosdv_sensor_kit"/>b
     <xacro:property name="sensor_kit_base_link" default="sensor_kit_base_link"/>
     <joint name="${sensor_kit_base_link}_joint" type="fixed">
@@ -141,4 +141,125 @@
       />
     </xacro:zed_camera>
+    <!-- USB Cameras -->
+    <!-- Front USB Camera -->
+    <joint name="usb_camera_front_joint" type="fixed">
+      <origin
+        xyz="${calibration['sensor_kit_base_link']['usb_camera_front']['x']}
+             ${calibration['sensor_kit_base_link']['usb_camera_front']['y']}
+             ${calibration['sensor_kit_base_link']['usb_camera_front']['z']}"
+        rpy="${calibration['sensor_kit_base_link']['usb_camera_front']['roll']}
+             ${calibration['sensor_kit_base_link']['usb_camera_front']['pitch']}
+             ${calibration['sensor_kit_base_link']['usb_camera_front']['yaw']}"
+      />
+      <parent link="sensor_kit_base_link"/>
+      <child link="usb_camera_front_link"/>
+    </joint>
+    <link name="usb_camera_front_link">
+      <visual>
+        <geometry>
+          <box size="0.03 0.08 0.03"/>
+        </geometry>
+        <material name="black">
+          <color rgba="0.1 0.1 0.1 1.0"/>
+        </material>
+      </visual>
+    </link>
+    <!-- Front camera optical frame -->
+    <joint name="usb_camera_front_optical_joint" type="fixed">
+      <origin xyz="0 0 0" rpy="-1.5708 0 -1.5708"/>
+      <parent link="usb_camera_front_link"/>
+      <child link="usb_camera_front_optical_link"/>
+    </joint>
+    <link name="usb_camera_front_optical_link"/>
+    <!-- Rear USB Camera -->
+    <joint name="usb_camera_rear_joint" type="fixed">
+      <origin
+        xyz="${calibration['sensor_kit_base_link']['usb_camera_rear']['x']}
+             ${calibration['sensor_kit_base_link']['usb_camera_rear']['y']}
+             ${calibration['sensor_kit_base_link']['usb_camera_rear']['z']}"
+        rpy="${calibration['sensor_kit_base_link']['usb_camera_rear']['roll']}
+             ${calibration['sensor_kit_base_link']['usb_camera_rear']['pitch']}
+             ${calibration['sensor_kit_base_link']['usb_camera_rear']['yaw']}"
+      />
+      <parent link="sensor_kit_base_link"/>
+      <child link="usb_camera_rear_link"/>
+    </joint>
+    <link name="usb_camera_rear_link">
+      <visual>
+        <geometry>
+          <box size="0.03 0.08 0.03"/>
+        </geometry>
+        <material name="black">
+          <color rgba="0.1 0.1 0.1 1.0"/>
+        </material>
+      </visual>
+    </link>
+    <!-- Rear camera optical frame -->
+    <joint name="usb_camera_rear_optical_joint" type="fixed">
+      <origin xyz="0 0 0" rpy="-1.5708 0 -1.5708"/>
+      <parent link="usb_camera_rear_link"/>
+      <child link="usb_camera_rear_optical_link"/>
+    </joint>
+    <link name="usb_camera_rear_optical_link"/>
+    <!-- Left USB Camera -->
+    <joint name="usb_camera_left_joint" type="fixed">
+      <origin
+        xyz="${calibration['sensor_kit_base_link']['usb_camera_left']['x']}
+             ${calibration['sensor_kit_base_link']['usb_camera_left']['y']}
+             ${calibration['sensor_kit_base_link']['usb_camera_left']['z']}"
+        rpy="${calibration['sensor_kit_base_link']['usb_camera_left']['roll']}
+             ${calibration['sensor_kit_base_link']['usb_camera_left']['pitch']}
+             ${calibration['sensor_kit_base_link']['usb_camera_left']['yaw']}"
+      />
+      <parent link="sensor_kit_base_link"/>
+      <child link="usb_camera_left_link"/>
+    </joint>
+    <link name="usb_camera_left_link">
+      <visual>
+        <geometry>
+          <box size="0.03 0.08 0.03"/>
+        </geometry>
+        <material name="black">
+          <color rgba="0.1 0.1 0.1 1.0"/>
+        </material>
+      </visual>
+    </link>
+    <!-- Left camera optical frame -->
+    <joint name="usb_camera_left_optical_joint" type="fixed">
+      <origin xyz="0 0 0" rpy="-1.5708 0 -1.5708"/>
+      <parent link="usb_camera_left_link"/>
+      <child link="usb_camera_left_optical_link"/>
+    </joint>
+    <link name="usb_camera_left_optical_link"/>
+    <!-- Right USB Camera -->
+    <joint name="usb_camera_right_joint" type="fixed">
+      <origin
+        xyz="${calibration['sensor_kit_base_link']['usb_camera_right']['x']}
+             ${calibration['sensor_kit_base_link']['usb_camera_right']['y']}
+             ${calibration['sensor_kit_base_link']['usb_camera_right']['z']}"
+        rpy="${calibration['sensor_kit_base_link']['usb_camera_right']['roll']}
+             ${calibration['sensor_kit_base_link']['usb_camera_right']['pitch']}
+             ${calibration['sensor_kit_base_link']['usb_camera_right']['yaw']}"
+      />
+      <parent link="sensor_kit_base_link"/>
+      <child link="usb_camera_right_link"/>
+    </joint>
+    <link name="usb_camera_right_link">
+      <visual>
+        <geometry>
+          <box size="0.03 0.08 0.03"/>
+        </geometry>
+        <material name="black">
+          <color rgba="0.1 0.1 0.1 1.0"/>
+        </material>
+      </visual>
+    </link>
+    <!-- Right camera optical frame -->
+    <joint name="usb_camera_right_optical_joint" type="fixed">
+      <origin xyz="0 0 0" rpy="-1.5708 0 -1.5708"/>
+      <parent link="usb_camera_right_link"/>
+      <child link="usb_camera_right_optical_link"/>
+    </joint>
+    <link name="usb_camera_right_optical_link"/>
   </xacro:macro>
 </robot>
