Commit message: Add selectable VLP16 LiDAR configuration

File: autosdv_sensor_kit_description/urdf/sensor_kit.xacro (robot description, xacro)
@@ -68,4 +68,24 @@
       </inertial>
     </link>
+    <!-- Velodyne VLP-16 LiDAR -->
+    <joint name="vlp16_joint" type="fixed">
+      <origin
+        xyz="${calibration['sensor_kit_base_link']['vlp16']['x']}
+             ${calibration['sensor_kit_base_link']['vlp16']['y']}
+             ${calibration['sensor_kit_base_link']['vlp16']['z']}"
+        rpy="${calibration['sensor_kit_base_link']['vlp16']['roll']}
+             ${calibration['sensor_kit_base_link']['vlp16']['pitch']}
+             ${calibration['sensor_kit_base_link']['vlp16']['yaw']}"
+      />
+      <parent link="sensor_kit_base_link"/>
+      <child link="vlp16"/>
+    </joint>
+    <link name="vlp16">
+      <inertial>
+        <mass value="0.1"/>
+        <origin xyz="0 0 0"/>
+        <inertia ixx="0.1" ixy="0" ixz="0" iyy="0.1" iyz="0" izz="0.1"/>
+      </inertial>
+    </link>
     <!-- Seyond Robin-W LiDAR -->
     <joint name="robin_w_joint" type="fixed">
